Commit message: fix body part

File: urdf/caster_body.urdf.xacro (robot description, xacro)
@@ -12,5 +12,5 @@
           <origin xyz="0 0 0" rpy="0 0 0" />
           <geometry>
-            <mesh filename="package://caster_body_description/mesh/caster_body_fixed.stl" />
+            <mesh filename="package://caster_description/mesh/caster_body_fixed.stl" />
           </geometry>
           <material name="">
@@ -23,6 +23,6 @@
         <origin xyz="0 0 0" rpy="0 0 0" />
         <geometry>
-          <mesh filename="package://caster_body_description/mesh/caster_body_part.stl" />
-          <!-- <mesh filename="package://caster_body_description/mesh/caster_body_part_up.stl" /> -->
+          <mesh filename="package://caster_description/mesh/caster_body_part.stl" />
+          <!-- <mesh filename="package://caster_description/mesh/caster_body_part_up.stl" /> -->
         </geometry>
         <material name="">
