Commit message: fix folder name, add v2 mesh and urdf

File: urdf/caster.urdf.xacro (robot description, xacro)
@@ -2,4 +2,5 @@
 <robot name="caster_robot" xmlns:xacro="http://www.ros.org/wiki/xacro" description="iqr caster robot">
   <xacro:property name="M_PI" value="3.1415926535897931" />
+  <xacro:include filename = "$(find caster_description)/urdf/common_properties.xacro" />
   <xacro:macro name="default_inertial" params="mass">
     <inertial>
@@ -16,5 +17,5 @@
         <origin xyz="0 0 0" rpy="0 0 0" />
         <geometry>
-          <mesh filename="package://caster_description/mesh/support_wheel.stl" />
+          <mesh filename="package://caster_description/mesh/v1/support_wheel.stl" />
         </geometry>
         <material name="">
@@ -38,5 +39,5 @@
         <origin xyz="0 0 0" rpy="0 0 ${invert*M_PI}" />
         <geometry>
-          <mesh filename="package://caster_description/mesh/drive_wheel.stl" />
+          <mesh filename="package://caster_description/mesh/v1/drive_wheel.stl" />
         </geometry>
         <material name="">
@@ -88,5 +89,5 @@
       <origin xyz="0 0 0" rpy="0 0 0" />
       <geometry>
-        <mesh filename="package://caster_description/mesh/caster_base.stl" />
+        <mesh filename="package://caster_description/mesh/v1/caster_base.stl" />
       </geometry>
       <material name="">

File: urdf/caster_xacro.xacro (robot description, xacro)
@@ -3,6 +3,5 @@
   <!-- Include accessories -->
   <xacro:include filename = "$(find caster_description)/urdf/common_properties.xacro" />
-  <xacro:include filename = "$(find caster_description)/urdf/iqr_caster.urdf.xacro" />
-  <xacro:include filename = "$(find caster_description)/urdf/iqr_caster.gazebo.xacro" />
+  <xacro:include filename = "$(find caster_description)/urdf/caster.urdf.xacro" />
   <xacro:caster/>
 </robot>

File: urdf/common_properties.xacro (robot description, xacro)
@@ -1,4 +1,4 @@
 <?xml version="1.0" ?>
-<robot name="xacro_properties" xmlns:xacro="http://ros.org/wiki/xacro">
+<robot name="xacro_properties" xmlns:xacro="http://www.ros.org/wiki/xacro">
   <!-- Init colour -->
   <material name="black">
