Commit message: fix incorrect v2 urdf include

File: urdf/caster_v2_gazebo.urdf.xacro (robot description, xacro)
@@ -2,5 +2,5 @@
 <robot name="caster_robot" xmlns:xacro="http://www.ros.org/wiki/xacro" description="iqr caster robot">
   <xacro:property name="M_PI" value="3.1415926535897931" />
-	<xacro:property name="deg_to_rad" value="0.017453293" />
+  <xacro:property name="deg_to_rad" value="0.017453293" />
   <!-- <xacro:include filename = "$(find caster_description)/urdf/common_properties.xacro" /> -->
   <xacro:include filename = "$(find caster_description)/urdf/iqr_caster.gazebo.xacro" />
@@ -55,5 +55,5 @@
       </inertial>
     </link>
-    <joint name="support_wheel_${location}_body_joint" type="fixed">
+    <joint name="support_wheel_${location}_body_joint" type="continuous">
       <xacro:insert_block name="origin" />
       <parent link="${parent}" />
@@ -62,5 +62,5 @@
       <dynamics damping="0.01" friction="0.0"/>
     </joint>
-    <joint name="support_wheel_${location}_joint" type="fixed">
+    <joint name="support_wheel_${location}_joint" type="continuous">
       <origin xyz="-0.0292 0 -0.0615" rpy="0 0 0" />
       <parent link="support_wheel_${location}_body_link" />

File: urdf/caster_v2_xacro.xacro (robot description, xacro)
@@ -4,4 +4,4 @@
   <xacro:include filename = "$(find caster_description)/urdf/common_properties.xacro" />
   <xacro:include filename = "$(find caster_description)/urdf/caster_v2.urdf.xacro" />
-  <xacro:caster/>
+  <!-- <xacro:caster_v2/>     -->
 </robot>

File: urdf/common_properties.xacro (robot description, xacro)
@@ -7,7 +7,4 @@
   <material name="dark">
     <color rgba="0.3 0.3 0.3 1.0"/>
-  </material>
-  <material name="light_black">
-    <color rgba="0.4 0.4 0.4 1.0"/>
   </material>
   <material name="blue">
