Commit message: gazebo config changed

File: urdf/caster_v2.urdf.xacro (robot description, xacro)
@@ -2,5 +2,7 @@
 <robot name="caster_robot" xmlns:xacro="http://www.ros.org/wiki/xacro" description="iqr caster robot">
   <xacro:property name="M_PI" value="3.1415926535897931" />
+	<xacro:property name="deg_to_rad" value="0.017453293" />
   <xacro:include filename = "$(find caster_description)/urdf/common_properties.xacro" />
+  <xacro:include filename = "$(find caster_description)/urdf/iqr_caster.gazebo.xacro" />
   <!-- support_wheel unit -->
   <xacro:macro name="support_wheel" params="parent location *origin">
@@ -22,9 +24,9 @@
       </collision>
       <inertial>
-        <origin xyz="-0.01 0 -0.02" />
+        <origin xyz="-0.01 0 -0.02" rpy="${24 * deg_to_rad} 0 ${M_PI/2}"/>
         <mass value="0.25" />
-        <inertia ixx="2.64583228e-4" ixy="0.0" ixz="-0.0"
-                 iyy="2.64583228e-4" iyz="0.0"
-                 izz="1.125e-4" />
+        <inertia ixx="2.4166657e-4" ixy="0.0" ixz="-0.0"
+                 iyy="2.4166657e-4" iyz="0.0"
+                 izz="6.66664e-5" />
       </inertial>
     </link>
@@ -46,9 +48,9 @@
       </collision>
       <inertial>
-        <origin xyz="0 0 0" />
-        <mass value="0.027" />
-        <inertia ixx="0.001" ixy="0.0" ixz="0.0"
-                 iyy="0.001" iyz="0.0"
-                 izz="0.001" />
+        <origin xyz="0 0 0" rpy="${M_PI/2} 0 0"/>
+        <mass value="0.27" />
+        <inertia ixx="7.35468456e-5" ixy="0.0" ixz="0.0"
+                 iyy="7.35468456e-5" iyz="0.0"
+                 izz="1.4259375e-4" />
       </inertial>
     </link>
@@ -58,5 +60,5 @@
       <child link="support_wheel_${location}_body_link" />
       <axis xyz="0 0 1" />
-      <dynamics damping="0.3" friction="0.0"/>
+      <dynamics damping="0.01" friction="0.0"/>
     </joint>
     <joint name="support_wheel_${location}_joint" type="continuous">
@@ -65,6 +67,4 @@
       <child link="support_wheel_${location}_link" />
       <axis xyz="0 1 0" />
-      <dynamics damping="0.3" friction="0.0"/>
-      <!-- <limit effort="10" velocity="10.0" /> -->
     </joint>
   </xacro:macro>
@@ -88,5 +88,5 @@
       </collision>
       <inertial>
-        <origin xyz="0 0 0" />
+        <origin xyz="0 0 0" rpy="${M_PI/2} 0 0"/>
         <mass value="0.92" />
         <inertia ixx="0.0014" ixy="0.0" ixz="-0.0"
@@ -100,6 +100,4 @@
       <child link="drive_wheel_${location}_link" />
       <axis xyz="0 1 0" rpy="0 0 0"/>
-      <dynamics damping="1.0" friction="0.0"/>
-      <!-- <limit effort="10" velocity="10.0" /> -->
     </joint>
     <transmission name="tran_${location}">
@@ -149,7 +147,7 @@
     </visual>
     <collision>
-      <origin xyz="0 0 0.135" rpy="0 0 0" />
+      <origin xyz="0 0 0.265" rpy="0 0 0" />
       <geometry>
-         <cylinder length="0.27" radius="0.275"/>
+         <cylinder length="0.005" radius="0.275"/>
       </geometry>
     </collision>
@@ -157,5 +155,5 @@
       <origin xyz="-0.02 0 0.11" />
       <mass value="45.16" />
-      <inertia ixx="0.94" ixy="0.01" ixz="0.03"
+      <inertia ixx="0.94" ixy="0.0" ixz="0.0"
            iyy="0.99" iyz="0.0"
            izz="1.35" />

Commit message: add top plate

File: urdf/caster_v2.urdf.xacro (robot description, xacro)
@@ -165,4 +165,10 @@
     <child link="base_link" />
   </joint>
+  <link name="top_plate_link" />
+  <joint name="top_plate_joint" type="fixed">
+    <origin xyz="0 0 0.266" rpy="0 0 0" />
+    <parent link="base_link" />
+    <child link="top_plate_link" />
+  </joint>
   <!-- IMU link -->
   <link name="imu_link" />
